Commit message: Further split and refactor sirius_description

File: src/sirius_description/urdf/materials.urdf.xacro (robot description, xacro)
@@ -4,7 +4,5 @@
   <material name="dark_bronze"> <color rgba=".36 .29 .22 1" /></material>
   <material name="dark_gray">   <color rgba="0.35 0.35 0.35 1"/></material>
-  <material name="gold">        <color rgba=".910 .443 .031 1" /></material>
   <material name="gray">        <color rgba=".796 .824 .937 1" /></material>
-  <material name="green">       <color rgba="0 1 0 1" /></material>
   <material name="white">       <color rgba="1 1 1 1" /></material>
   <!-- Gazebo colors -->
@@ -33,12 +31,4 @@
     </material>
   </xacro:macro>
-  <xacro:macro name="gold">
-    <material>
-      <ambient>1 .6 .2 1</ambient>
-      <diffuse>1 .6 .2 1</diffuse>
-      <specular>.4 .2 .1 1</specular>
-      <emissive>0.0 0.0 0.0 0.0</emissive>
-    </material>
-  </xacro:macro>
   <xacro:macro name="gray">
     <material>
@@ -46,12 +36,4 @@
       <diffuse>0.92 0.95 1 1</diffuse>
       <specular>1 1 1 1</specular>
-      <emissive>0.0 0.0 0.0 0.0</emissive>
-    </material>
-  </xacro:macro>
-  <xacro:macro name="green">
-    <material>
-      <ambient>0 1 0 1</ambient>
-      <diffuse>0 1 0 1</diffuse>
-      <specular>0 0 0 1</specular>
       <emissive>0.0 0.0 0.0 0.0</emissive>
     </material>

File: src/sirius_description/urdf/sirius/gnss.urdf.xacro (robot description, xacro)
@@ -3,11 +3,12 @@
      https://www.sparkfun.com/products/21801 -->
 <robot xmlns:xacro="http://wiki.ros.org/xacro">
-<xacro:macro name="gnss" params="material package:=^ collisions:=^ inertial:=^ datum:=^ elevation:=^">
-  <link name="gnss">
+<xacro:macro name="gnss" params="prefix:='' material collisions:=${xacro.load_yaml('$(find sirius_description)/urdf/sirius/collisions.yaml')} inertial:=${xacro.load_yaml('$(find sirius_description)/config/inertial/gnss.yaml')} datum:=^ elevation:=^ horizontal_cep:=1.0 vertical_cep:=1.5 rate:=20.0">
+  <xacro:property name="_prefix" value="${prefix + '_' if prefix else ''}"/>
+  <link name="${_prefix}gnss">
     <visual>
       <material name="${material}">
       </material>
       <geometry>
-        <mesh filename="package://${package}/meshes/sirius/gnss.stl" scale="0.001 0.001 0.001"/>
+        <mesh filename="package://sirius_description/meshes/sirius/gnss.stl" scale="0.001 0.001 0.001"/>
       </geometry>
       <origin xyz="0 0 ${collisions['gnss_height']/2}" rpy="${pi/2} 0 0" />
@@ -24,5 +25,5 @@
     </collision>
   </link>
-  <gazebo reference="gnss">
+  <gazebo reference="${_prefix}gnss">
     <sensor type="gps" name="gps_sensor">
       <always_on>true</always_on>
@@ -32,6 +33,7 @@
           <horizontal>
             <noise type="gaussian">
-              <mean>0.0</mean>
-              <stddev>0.03</stddev>
+              <!-- sqrt(-1/(2*log(0.5))) = 0.8493218002880191 -->
+              <!-- This is the ratio needed to convert CEP to std dev of single axis -->
+              <stddev>${horizontal_cep * 0.8493218002880191}</stddev>
             </noise>
           </horizontal>
@@ -39,5 +41,5 @@
             <noise type="gaussian">
               <mean>0.0</mean>
-              <stddev>0.03</stddev>
+              <stddev>${vertical_cep * 0.8493218002880191}</stddev>
             </noise>
           </vertical>
@@ -46,12 +48,10 @@
           <horizontal>
             <noise type="gaussian">
-              <mean>0.0</mean>
-              <stddev>0.05</stddev>
+              <stddev>${0.05 * 0.8493218002880191}</stddev>
             </noise>
           </horizontal>
           <vertical>
             <noise type="gaussian">
-              <mean>0.0</mean>
-              <stddev>0.05</stddev>
+              <stddev>${0.05 * 0.8493218002880191}</stddev>
             </noise>
           </vertical>
@@ -61,5 +61,5 @@
         <topicName>/gps/fix</topicName>
         <frameName>gnss</frameName>
-        <updateRateHZ>20.0</updateRateHZ>
+        <updateRateHZ>${rate}</updateRateHZ>
         <sphericalCoordinates>
             <latitudeDeg>${datum[0]}</latitudeDeg>
@@ -68,10 +68,10 @@
             <elevation>${elevation}</elevation>
         </sphericalCoordinates>
-        <positionCovariance>0.03 0 0 0 0.03 0 0 0 0.03</positionCovariance>
+        <positionCovariance>${horizontal_cep * 0.8493218002880191} 0 0 0 ${horizontal_cep * 0.8493218002880191} 0 0 0 ${vertical_cep * 0.8493218002880191}</positionCovariance>
         <positionCovarianceType>diagonal_known</positionCovarianceType>
       </plugin>
     </sensor>
   </gazebo>
-  <gazebo reference="gnss">
+  <gazebo reference="${_prefix}gnss">
       <visual>
         <xacro:element xacro:name="xacro:${material}" />

File: src/sirius_description/urdf/sirius/indicator_light.urdf.xacro (robot description, xacro)
@@ -1,11 +1,12 @@
 <?xml version="1.0" encoding="utf-8"?>
 <robot xmlns:xacro="http://wiki.ros.org/xacro">
-<xacro:macro name="indicator_light" params="material prefix:='' package:=^ collisions:=^ inertial:=^">
-  <link name="${prefix + '_' if prefix else prefix}indicator_light">
+<xacro:macro name="indicator_light" params="material prefix:='' collisions:=${xacro.load_yaml('$(find sirius_description)/urdf/sirius/collisions.yaml')} inertial:=${xacro.load_yaml('$(find sirius_description)/config/inertial/indicator_light.yaml')}">
+  <xacro:property name="_prefix" value="${prefix + '_' if prefix else ''}"/>
+  <link name="${_prefix}indicator_light">
     <visual>
       <material name="${material}">
       </material>
       <geometry>
-        <mesh filename="package://${package}/meshes/sirius/indicator_light.stl" scale="0.001 0.001 0.001"/>
+        <mesh filename="package://sirius_description/meshes/sirius/indicator_light.stl" scale="0.001 0.001 0.001"/>
       </geometry>
     </visual>
@@ -21,5 +22,5 @@
     </collision>
   </link>
-  <gazebo reference="${prefix + '_' if prefix else prefix}indicator_light">
+  <gazebo reference="${_prefix}indicator_light">
       <visual>
         <xacro:element xacro:name="xacro:${material}" />

File: src/sirius_description/urdf/sirius/platform.urdf.xacro (robot description, xacro)
@@ -1,71 +1,72 @@
 <robot xmlns:xacro="http://wiki.ros.org/xacro">
-<xacro:macro name="platform" params="material prefix:=''  package:=^ collisions:=^ params:=^ inertial:=^">
-    <link name="${prefix + '_' if prefix else prefix}platform">
-      <visual>
-        <material name="${material}"/>
-        <geometry>
-        <mesh filename="package://${package}/meshes/sirius/platform.stl" scale="0.001 0.001 0.001"/>
-        </geometry>
-      </visual>
-      <inertial>
-        <origin xyz="0 0 0" rpy="0 0 ${pi}"/>
-        <mass value="${inertial['platform_mass']}"/>
-        <inertia ixx="${inertial['platform_inertia']['ixx']}" ixy="${inertial['platform_inertia']['ixy']}" ixz="${inertial['platform_inertia']['ixz']}" iyy="${inertial['platform_inertia']['iyy']}" iyz="${inertial['platform_inertia']['iyz']}" izz="${inertial['platform_inertia']['izz']}"/>
-      </inertial>
-      <collision>
-        <geometry>
-          <box size="${collisions['platform_box_length']} ${params['suspension_separation_y'] - collisions['suspension_thickness']*1.5} ${collisions['platform_height']}"/>
-        </geometry>
-        <origin xyz="${collisions['platform_box_x']} 0 ${collisions['platform_height']/2}" />
-      </collision>
-      <collision>
-        <geometry>
-          <box size="${collisions['platform_height']/tan(collisions['platform_angle'] * pi / 180) - collisions['platform_profile_size']} ${params['suspension_separation_y'] - collisions['suspension_thickness']*1.5} ${collisions['platform_profile_size']}"/>
-        </geometry>
-        <origin xyz="${collisions['platform_height']/(tan(collisions['platform_angle'] * pi / 180)*2) - collisions['platform_profile_size']/2 + collisions['platform_box_x'] + collisions['platform_box_length']/2} 0 ${collisions['platform_height'] - collisions['platform_profile_size']/2}" />
-      </collision>
-      <collision>
-        <geometry>
-          <box size="${collisions['platform_height']/cos(collisions['platform_angle'] * pi / 180) - collisions['platform_profile_size']/2} ${collisions['platform_profile_size']} ${collisions['platform_profile_size']}"/>
-        </geometry>
-        <origin xyz="${collisions['platform_box_x'] + collisions['platform_box_length']/2 + collisions['platform_height']/(tan(collisions['platform_angle'] * pi / 180) * 2) - collisions['platform_profile_size']/2} ${params['suspension_separation_y']/2 - collisions['platform_profile_size']*1.8} ${collisions['platform_height']/2 + collisions['platform_profile_size']/6}" rpy="0 ${-collisions['platform_angle'] * pi / 180} 0"/>
-      </collision>
-      <collision>
-        <geometry>
-          <box size="${collisions['platform_height']/cos(collisions['platform_angle'] * pi / 180) - collisions['platform_profile_size']/2} ${collisions['platform_profile_size']} ${collisions['platform_profile_size']}"/>
-        </geometry>
-        <origin xyz="${collisions['platform_box_x'] + collisions['platform_box_length']/2 + collisions['platform_height']/(tan(collisions['platform_angle'] * pi / 180) * 2) - collisions['platform_profile_size']/2} ${-params['suspension_separation_y']/2 + collisions['platform_profile_size']*1.8} ${collisions['platform_height']/2 + collisions['platform_profile_size']/6}" rpy="0 ${-collisions['platform_angle'] * pi / 180} 0"/>
-      </collision>
-      <collision>
-        <geometry>
-        <!-- ${collisions['platform_mast_radius']} -->
-          <box size="${collisions['platform_profile_size']} ${collisions['platform_profile_size']} ${collisions['platform_mast_height']}"/>
-        </geometry>
-        <origin xyz="${collisions['platform_mast_x']} ${collisions['platform_mast_y']} ${collisions['platform_mast_height']/2}" />
-      </collision>
-      <collision>
-        <geometry>
-          <box size="${collisions['platform_profile_size']} ${collisions['platform_profile_size']} ${collisions['platform_mast_height']}"/>
-        </geometry>
-        <origin xyz="${collisions['platform_mast_x']} ${-collisions['platform_mast_y']} ${collisions['platform_mast_height']/2}" />
-      </collision>
-      <collision>
-        <geometry>
-          <box size="${collisions['platform_profile_size']} ${collisions['platform_mast_y']*2} ${collisions['platform_profile_size']}"/>
-        </geometry>
-        <origin xyz="${collisions['platform_mast_x']} 0 ${collisions['platform_mast_height'] - collisions['platform_profile_size']*2.55}" />
-      </collision>
-      <collision>
-        <geometry>
-          <cylinder length="${collisions['platform_mast_5g_length']}" radius="${collisions['platform_mast_5g_radius']}"/>
-        </geometry>
-        <origin xyz="${collisions['platform_mast_5g_xyz']}" />
-      </collision>
-    </link>
-    <gazebo reference="${prefix + '_' if prefix else prefix}platform">
-      <visual>
-        <xacro:element xacro:name="xacro:${material}" />
-      </visual>
-    </gazebo>
+<xacro:macro name="platform" params="material prefix:='' collisions:=${xacro.load_yaml('$(find sirius_description)/urdf/sirius/collisions.yaml')} inertial:=${xacro.load_yaml('$(find sirius_description)/config/inertial/platform.yaml')} mechanical:=${xacro.load_yaml('$(find sirius_description)/config/mechanical.yaml')}">
+  <xacro:property name="_prefix" value="${prefix + '_' if prefix else ''}"/>
+  <link name="${_prefix}platform">
+    <visual>
+      <material name="${material}"/>
+      <geometry>
+      <mesh filename="package://sirius_description/meshes/sirius/platform.stl" scale="0.001 0.001 0.001"/>
+      </geometry>
+    </visual>
+    <inertial>
+      <origin xyz="0 0 0" rpy="0 0 ${pi}"/>
+      <mass value="${inertial['platform_mass']}"/>
+      <inertia ixx="${inertial['platform_inertia']['ixx']}" ixy="${inertial['platform_inertia']['ixy']}" ixz="${inertial['platform_inertia']['ixz']}" iyy="${inertial['platform_inertia']['iyy']}" iyz="${inertial['platform_inertia']['iyz']}" izz="${inertial['platform_inertia']['izz']}"/>
+    </inertial>
+    <collision>
+      <geometry>
+        <box size="${collisions['platform_box_length']} ${mechanical['suspension_separation_y'] - collisions['suspension_thickness']*1.5} ${collisions['platform_height']}"/>
+      </geometry>
+      <origin xyz="${collisions['platform_box_x']} 0 ${collisions['platform_height']/2}" />
+    </collision>
+    <collision>
+      <geometry>
+        <box size="${collisions['platform_height']/tan(collisions['platform_angle'] * pi / 180) - collisions['platform_profile_size']} ${mechanical['suspension_separation_y'] - collisions['suspension_thickness']*1.5} ${collisions['platform_profile_size']}"/>
+      </geometry>
+      <origin xyz="${collisions['platform_height']/(tan(collisions['platform_angle'] * pi / 180)*2) - collisions['platform_profile_size']/2 + collisions['platform_box_x'] + collisions['platform_box_length']/2} 0 ${collisions['platform_height'] - collisions['platform_profile_size']/2}" />
+    </collision>
+    <collision>
+      <geometry>
+        <box size="${collisions['platform_height']/cos(collisions['platform_angle'] * pi / 180) - collisions['platform_profile_size']/2} ${collisions['platform_profile_size']} ${collisions['platform_profile_size']}"/>
+      </geometry>
+      <origin xyz="${collisions['platform_box_x'] + collisions['platform_box_length']/2 + collisions['platform_height']/(tan(collisions['platform_angle'] * pi / 180) * 2) - collisions['platform_profile_size']/2} ${mechanical['suspension_separation_y']/2 - collisions['platform_profile_size']*1.8} ${collisions['platform_height']/2 + collisions['platform_profile_size']/6}" rpy="0 ${-collisions['platform_angle'] * pi / 180} 0"/>
+    </collision>
+    <collision>
+      <geometry>
+        <box size="${collisions['platform_height']/cos(collisions['platform_angle'] * pi / 180) - collisions['platform_profile_size']/2} ${collisions['platform_profile_size']} ${collisions['platform_profile_size']}"/>
+      </geometry>
+      <origin xyz="${collisions['platform_box_x'] + collisions['platform_box_length']/2 + collisions['platform_height']/(tan(collisions['platform_angle'] * pi / 180) * 2) - collisions['platform_profile_size']/2} ${-mechanical['suspension_separation_y']/2 + collisions['platform_profile_size']*1.8} ${collisions['platform_height']/2 + collisions['platform_profile_size']/6}" rpy="0 ${-collisions['platform_angle'] * pi / 180} 0"/>
+    </collision>
+    <collision>
+      <geometry>
+      <!-- ${collisions['platform_mast_radius']} -->
+        <box size="${collisions['platform_profile_size']} ${collisions['platform_profile_size']} ${collisions['platform_mast_height']}"/>
+      </geometry>
+      <origin xyz="${collisions['platform_mast_x']} ${collisions['platform_mast_y']} ${collisions['platform_mast_height']/2}" />
+    </collision>
+    <collision>
+      <geometry>
+        <box size="${collisions['platform_profile_size']} ${collisions['platform_profile_size']} ${collisions['platform_mast_height']}"/>
+      </geometry>
+      <origin xyz="${collisions['platform_mast_x']} ${-collisions['platform_mast_y']} ${collisions['platform_mast_height']/2}" />
+    </collision>
+    <collision>
+      <geometry>
+        <box size="${collisions['platform_profile_size']} ${collisions['platform_mast_y']*2} ${collisions['platform_profile_size']}"/>
+      </geometry>
+      <origin xyz="${collisions['platform_mast_x']} 0 ${collisions['platform_mast_height'] - collisions['platform_profile_size']*2.55}" />
+    </collision>
+    <collision>
+      <geometry>
+        <cylinder length="${collisions['platform_mast_5g_length']}" radius="${collisions['platform_mast_5g_radius']}"/>
+      </geometry>
+      <origin xyz="${collisions['platform_mast_5g_xyz']}" />
+    </collision>
+  </link>
+  <gazebo reference="${_prefix}platform">
+    <visual>
+      <xacro:element xacro:name="xacro:${material}" />
+    </visual>
+  </gazebo>
 </xacro:macro>
 </robot>

File: src/sirius_description/urdf/sirius/rim.urdf.xacro (robot description, xacro)
@@ -1,30 +1,31 @@
 <robot xmlns:xacro="http://wiki.ros.org/xacro">
-<xacro:macro name="rim" params="prefix material package:=^ params:=^">
-    <link name="${prefix}_rim">
-      <visual>
-        <material name="${material}" />
-        <geometry>
-          <mesh filename="package://${package}/meshes/sirius/rim.stl" scale="0.001 0.001 0.001"/>
-        </geometry>
-      </visual>
-      <!-- Without inertia link is either lumped with parent or removed from sdf -->
-      <!-- Link cannot be lumped with parent If we want to apply different material to it -->
-      <!-- Zero inertia is not allowed, so we use very small values as a workaround -->
-      <inertial>
-        <mass value="1e-5"/>
-        <inertia ixx="1e-9" ixy="1e-9" ixz="1e-9" iyy="1e-9" iyz="1e-9" izz="1e-9"/>
-      </inertial>
-      <collision>
-        <geometry>
-          <cylinder length="${params['rim_width']}" radius="${params['wheel_radius'] * 0.8}"/>
-        </geometry>
-        <origin xyz="0 0 0" rpy="${pi/2} 0 0" />
-      </collision>
-    </link>
-    <gazebo reference="${prefix}_wheel_rim">
-      <visual>
-        <xacro:element xacro:name="xacro:${material}" />
-      </visual>
-    </gazebo>
+<xacro:macro name="rim" params="prefix:='' material mechanical:=${xacro.load_yaml('$(find sirius_description)/config/mechanical.yaml')}">
+  <xacro:property name="_prefix" value="${prefix + '_' if prefix else ''}"/>
+  <link name="${_prefix}rim">
+    <visual>
+      <material name="${material}" />
+      <geometry>
+        <mesh filename="package://sirius_description/meshes/sirius/rim.stl" scale="0.001 0.001 0.001"/>
+      </geometry>
+    </visual>
+    <!-- Without inertia link is either lumped with parent or removed from sdf -->
+    <!-- Link cannot be lumped with parent If we want to apply different material to it -->
+    <!-- Zero inertia is not allowed, so we use very small values as a workaround -->
+    <inertial>
+      <mass value="1e-5"/>
+      <inertia ixx="1e-9" ixy="1e-9" ixz="1e-9" iyy="1e-9" iyz="1e-9" izz="1e-9"/>
+    </inertial>
+    <collision>
+      <geometry>
+        <cylinder length="${mechanical['rim_width']}" radius="${mechanical['wheel_radius'] * 0.8}"/>
+      </geometry>
+      <origin xyz="0 0 0" rpy="${pi/2} 0 0" />
+    </collision>
+  </link>
+  <gazebo reference="${_prefix}rim">
+    <visual>
+      <xacro:element xacro:name="xacro:${material}" />
+    </visual>
+  </gazebo>
 </xacro:macro>
 </robot>

File: src/sirius_description/urdf/sirius/suspension.urdf.xacro (robot description, xacro)
@@ -1,28 +1,29 @@
 <robot xmlns:xacro="http://wiki.ros.org/xacro">
-<xacro:macro name="suspension" params="prefix material flip:=false params:=^ package:=^ collisions:=^ inertial:=^">
-    <link name="${prefix}_suspension">
-      <visual>
-        <material name="${material}"/>
-        <geometry>
-          <mesh filename="package://${package}/meshes/sirius/suspension.stl" scale="0.001 0.001 0.001"/>
-        </geometry>
-        <origin xyz="0 0 0" rpy="0 0 ${pi if flip else 0}" />
-      </visual>
-      <inertial>
-        <mass value="${inertial['suspension_mass']}"/>
-        <inertia ixx="${inertial['suspension_inertia']['ixx']}" ixy="${inertial['suspension_inertia']['ixy']}" ixz="${inertial['suspension_inertia']['ixz']}" iyy="${inertial['suspension_inertia']['iyy']}" iyz="${inertial['suspension_inertia']['iyz']}" izz="${inertial['suspension_inertia']['izz']}"/>
-      </inertial>
-      <collision>
-        <geometry>
-          <box size="${collisions['suspension_width']} ${collisions['suspension_thickness']} ${collisions['suspension_length']}"/>
-        </geometry>
-        <origin xyz="${(1 - 2 * flip) * (params['wheel_base']/4 - params['suspension_separation_x']/4 + collisions['suspension_x_shift'])} 0 ${-params['suspension_height']/2}" rpy="0 ${collisions['suspension_angle'] * pi / 180} ${pi if flip else 0}" />
-      </collision>
-    </link>
-    <gazebo reference="${prefix}_suspension">
-      <visual>
-        <xacro:element xacro:name="xacro:${material}" />
-      </visual>
-    </gazebo>
+<xacro:macro name="suspension" params="prefix:='' material flip:=false mechanical:=${xacro.load_yaml('$(find sirius_description)/config/mechanical.yaml')} collisions:=${xacro.load_yaml('$(find sirius_description)/urdf/sirius/collisions.yaml')} inertial:=${xacro.load_yaml('$(find sirius_description)/config/inertial/suspension.yaml')}">
+  <xacro:property name="_prefix" value="${prefix + '_' if prefix else ''}"/>
+  <link name="${_prefix}suspension">
+    <visual>
+      <material name="${material}"/>
+      <geometry>
+        <mesh filename="package://sirius_description/meshes/sirius/suspension.stl" scale="0.001 0.001 0.001"/>
+      </geometry>
+      <origin xyz="0 0 0" rpy="0 0 ${pi if flip else 0}" />
+    </visual>
+    <inertial>
+      <mass value="${inertial['suspension_mass']}"/>
+      <inertia ixx="${inertial['suspension_inertia']['ixx']}" ixy="${inertial['suspension_inertia']['ixy']}" ixz="${inertial['suspension_inertia']['ixz']}" iyy="${inertial['suspension_inertia']['iyy']}" iyz="${inertial['suspension_inertia']['iyz']}" izz="${inertial['suspension_inertia']['izz']}"/>
+    </inertial>
+    <collision>
+      <geometry>
+        <box size="${collisions['suspension_width']} ${collisions['suspension_thickness']} ${collisions['suspension_length']}"/>
+      </geometry>
+      <origin xyz="${(1 - 2 * flip) * (mechanical['wheel_base']/4 - mechanical['suspension_separation_x']/4 + collisions['suspension_x_shift'])} 0 ${-mechanical['suspension_height']/2}" rpy="0 ${collisions['suspension_angle'] * pi / 180} ${pi if flip else 0}" />
+    </collision>
+  </link>
+  <gazebo reference="${_prefix}suspension">
+    <visual>
+      <xacro:element xacro:name="xacro:${material}" />
+    </visual>
+  </gazebo>
 </xacro:macro>
 </robot>
