Commit message: Further split and refactor sirius_description

File: src/sirius_description/urdf/sirius/wheel.urdf.xacro (robot description, xacro)
@@ -1,51 +1,52 @@
 <robot xmlns:xacro="http://wiki.ros.org/xacro">
 <xacro:include filename="rim.urdf.xacro" />
-<xacro:macro name="wheel" params="prefix material material_rim flip:=false package:=^ params:=^ inertial:=^">
-    <link name="${prefix}_wheel">
-      <visual>
-        <material name="${material}" />
-        <geometry>
-          <mesh filename="package://${package}/meshes/sirius/wheel.stl" scale="0.001 0.001 0.001"/>
-        </geometry>
-        <origin xyz="0 0 0" />
-      </visual>
-      <inertial>
-        <origin xyz="0 ${-params['wheel_width']/2} 0" />
-        <mass value="${inertial['wheel_mass']}"/>
-        <inertia ixx="${inertial['wheel_inertia']['ixx']}" ixy="${inertial['wheel_inertia']['ixy']}" ixz="${inertial['wheel_inertia']['ixz']}" iyy="${inertial['wheel_inertia']['iyy']}" iyz="${inertial['wheel_inertia']['iyz']}" izz="${inertial['wheel_inertia']['izz']}"/>
-      </inertial>
-      <collision>
-        <geometry>
-          <cylinder length="${params['wheel_width']}" radius="${params['wheel_radius']}"/>
-        </geometry>
-        <origin xyz="0 0 0" rpy="${pi/2} 0 0" />
-      </collision>
-    </link>
-    <xacro:rim prefix="${prefix}_wheel_outside" material="${material_rim}" />
-    <xacro:rim prefix="${prefix}_wheel_inside" material="${material_rim}" />
-    <joint name="${prefix}_wheel_to_outside_rim_joint" type="fixed">
-      <parent link="${prefix}_wheel"/>
-      <child link="${prefix}_wheel_outside_rim"/>
-      <origin xyz="0 ${ (1 - 2*flip) * (params['wheel_width'] + params['rim_width'])/2} 0" />
-    </joint>
-    <joint name="${prefix}_wheel_to_inside_rim_joint" type="fixed">
-      <parent link="${prefix}_wheel"/>
-      <child link="${prefix}_wheel_inside_rim"/>
-      <origin xyz="0 ${ (2*flip - 1) * (params['wheel_width'] + params['rim_width'])/2} 0" />
-    </joint>
-    <gazebo reference="${prefix}_wheel">
-      <visual>
-        <xacro:element xacro:name="xacro:${material}" />
-      </visual>
-    </gazebo>
-    <!-- This is required so wheel and rim link are not lumped together -->
-    <!-- Otherwise, they would be given the same material (color) during urdf->sdf conversion -->
-    <!-- Possibly, in future versions of gazebo, we could apply different materials to different visual elements in URDF -->
-    <gazebo reference="${prefix}_wheel_to_outside_rim_joint">
-      <preserveFixedJoint>true</preserveFixedJoint>
-    </gazebo>
-    <gazebo reference="${prefix}_wheel_to_inside_rim_joint">
-      <preserveFixedJoint>true</preserveFixedJoint>
-    </gazebo>
+<xacro:macro name="wheel" params="prefix:='' material material_rim flip:=false mechanical:=${xacro.load_yaml('$(find sirius_description)/config/mechanical.yaml')} inertial:=${xacro.load_yaml('$(find sirius_description)/config/inertial/wheel.yaml')}">
+  <xacro:property name="_prefix" value="${prefix + '_' if prefix else ''}"/>
+  <link name="${_prefix}wheel">
+    <visual>
+      <material name="${material}" />
+      <geometry>
+        <mesh filename="package://sirius_description/meshes/sirius/wheel.stl" scale="0.001 0.001 0.001"/>
+      </geometry>
+      <origin xyz="0 0 0" />
+    </visual>
+    <inertial>
+      <origin xyz="0 ${-mechanical['wheel_width']/2} 0" />
+      <mass value="${inertial['wheel_mass']}"/>
+      <inertia ixx="${inertial['wheel_inertia']['ixx']}" ixy="${inertial['wheel_inertia']['ixy']}" ixz="${inertial['wheel_inertia']['ixz']}" iyy="${inertial['wheel_inertia']['iyy']}" iyz="${inertial['wheel_inertia']['iyz']}" izz="${inertial['wheel_inertia']['izz']}"/>
+    </inertial>
+    <collision>
+      <geometry>
+        <cylinder length="${mechanical['wheel_width']}" radius="${mechanical['wheel_radius']}"/>
+      </geometry>
+      <origin xyz="0 0 0" rpy="${pi/2} 0 0" />
+    </collision>
+  </link>
+  <xacro:rim prefix="${_prefix}outer" material="${material_rim}" />
+  <xacro:rim prefix="${_prefix}inner" material="${material_rim}" />
+  <joint name="${_prefix}outer_rim_joint" type="fixed">
+    <parent link="${_prefix}wheel"/>
+    <child link="${_prefix}outer_rim"/>
+    <origin xyz="0 ${ (1 - 2*flip) * (mechanical['wheel_width'] + mechanical['rim_width'])/2} 0" />
+  </joint>
+  <joint name="${_prefix}inner_rim_joint" type="fixed">
+    <parent link="${_prefix}wheel"/>
+    <child link="${_prefix}inner_rim"/>
+    <origin xyz="0 ${ (2*flip - 1) * (mechanical['wheel_width'] + mechanical['rim_width'])/2} 0" />
+  </joint>
+  <gazebo reference="${_prefix}wheel">
+    <visual>
+      <xacro:element xacro:name="xacro:${material}" />
+    </visual>
+  </gazebo>
+  <!-- This is required so wheel and rim link are not lumped together -->
+  <!-- Otherwise, they would be given the same material (color) during urdf->sdf conversion -->
+  <!-- Possibly, in future versions of gazebo, we could apply different materials to different visual elements in URDF -->
+  <gazebo reference="${_prefix}outer_rim_joint">
+    <preserveFixedJoint>true</preserveFixedJoint>
+  </gazebo>
+  <gazebo reference="${_prefix}inner_rim_joint">
+    <preserveFixedJoint>true</preserveFixedJoint>
+  </gazebo>
 </xacro:macro>
 </robot>
