Commit message: Refactor localization and tweak simulation

File: src/sirius_common/sirius_description/robots/sirius.urdf.xacro (robot description, xacro)
@@ -44,14 +44,14 @@
   </xacro:macro>
     <!-- Macro to combine suspension and wheel -->
-  <xacro:macro name="drive_system" params="prefix flip_x:=false flip_y:=false mechanical:=^">
-    <xacro:suspension prefix="${prefix}" material="dark_bronze" flip="${flip_y}" />
-    <xacro:wheel prefix="${prefix}" material="dark_gray" material_rim="white" flip="${flip_x}" />
+  <xacro:macro name="drive_system" params="prefix flip_y_plane:=false flip_x_plane:=false mechanical:=^">
+    <xacro:suspension prefix="${prefix}" material="dark_bronze" flip_x_plane="${flip_x_plane}" flip_y_plane="${flip_y_plane}" />
+    <xacro:wheel prefix="${prefix}" material="dark_gray" material_rim="white" flip="${flip_y_plane}" />
     <xacro:joint  type="continuous"
                   parent="${prefix}_suspension"
                   child="${prefix}_wheel"
-                  xyz="${(1 - 2 * flip_y)  * (mechanical['wheel_base'] - mechanical['suspension_separation_x'])/2 } ${(1 - 2 * flip_x)  * (mechanical['wheel_track'] - mechanical['suspension_separation_y'])/2} ${-mechanical['suspension_height']}"
+                  xyz="${(1 - 2 * flip_x_plane)  * (mechanical['wheel_base'] - mechanical['suspension_separation_x'])/2 } ${(1 - 2 * flip_y_plane)  * (mechanical['wheel_track'] - mechanical['suspension_separation_y'])/2} ${-mechanical['suspension_height']}"
                   rpy="0 0 0"
                   axis="0 1 0"
-                  limit_effort="18.0"
+                  limit_effort="80.0"
                   limit_velocity="8.0" />
     <transmission name="${prefix}_wheel_transmission">
@@ -68,8 +68,8 @@
   <link name="base_link" />
   <xacro:platform material="white" />
-  <xacro:drive_system prefix="back_left" flip_y="true" />
-  <xacro:drive_system prefix="back_right" flip_x="true" flip_y="true"/>
+  <xacro:drive_system prefix="back_left" flip_x_plane="true" />
+  <xacro:drive_system prefix="back_right" flip_y_plane="true" flip_x_plane="true"/>
   <xacro:drive_system prefix="front_left" />
-  <xacro:drive_system prefix="front_right"  flip_x="true"/>
+  <xacro:drive_system prefix="front_right"  flip_y_plane="true"/>
   <xacro:indicator_light material="gray" />
   <!-- Define sensors and cameras links -->

File: src/sirius_common/sirius_description/urdf/hp_4310/hp_4310.urdf.xacro (robot description, xacro)
@@ -1,4 +1,4 @@
 <robot xmlns:xacro="http://wiki.ros.org/xacro">
-<xacro:macro name="hp_4310" params="prefix:=hp_4310 material cameras:=${xacro.load_yaml('$(find sirius_description)/urdf/hp_4310/collisions.yaml')} cameras_inertial:=${xacro.load_yaml('$(find sirius_description)/config/inertial/hp_4310.yaml')}">
+<xacro:macro name="hp_4310" params="prefix:=hp_4310 material cameras:=${xacro.load_yaml('$(find sirius_description)/urdf/hp_4310/collisions.yaml')}">
   <link name="${prefix}_camera">
     <visual>
@@ -15,8 +15,4 @@
       <origin xyz="${-cameras['hp_4310_thickness']/2} 0 0"/>
     </collision>
-    <cameras_inertial>
-      <mass value="${cameras_inertial['hp_4310_mass']}"/>
-      <inertia ixx="${cameras_inertial['hp_4310_inertia']['ixx']}" ixy="${cameras_inertial['hp_4310_inertia']['ixy']}" ixz="${cameras_inertial['hp_4310_inertia']['ixz']}" iyy="${cameras_inertial['hp_4310_inertia']['iyy']}" iyz="${cameras_inertial['hp_4310_inertia']['iyz']}" izz="${cameras_inertial['hp_4310_inertia']['izz']}"/>
-    </cameras_inertial>
   </link>
   <gazebo reference="${prefix}_camera">

File: src/sirius_common/sirius_description/urdf/oak-d-w/oak-d-w.urdf.xacro (robot description, xacro)
@@ -1,7 +1,11 @@
 <?xml version="1.0"?>
 <robot xmlns:xacro="http://ros.org/wiki/xacro">
-<xacro:macro name="oak-d-w" params="prefix:=oak-d-w collisions:=${xacro.load_yaml('$(find sirius_description)/urdf/oak-d-w/collisions.yaml')} cameras_inertial:=${xacro.load_yaml('$(find sirius_description)/config/inertial/oak-d-w.yaml')} stereo_fps:=^|30 imu_frequency:=^|200 datum:=^ elevation:=^ year:=^ calibration:=${xacro.load_yaml('$(find sirius_calibration)/kalibr/camimu/inflated/camimu-camchain-imucam.yaml')} imu_calibration:=${xacro.load_yaml('$(find sirius_calibration)/kalibr/camimu/inflated/camimu-imu.yaml')}">
+<xacro:macro name="oak-d-w" params="prefix:=oak-d-w collisions:=${xacro.load_yaml('$(find sirius_description)/urdf/oak-d-w/collisions.yaml')} stereo_fps:=^|30 imu_frequency:=^|200 datum:=^ elevation:=^ year:=^ calibration:=${xacro.load_yaml('$(find sirius_calibration)/kalibr/camimu/inflated/camimu-camchain-imucam.yaml')} imu_calibration:=${xacro.load_yaml('$(find sirius_calibration)/kalibr/camimu/inflated/camimu-imu.yaml')}">
   <xacro:property name="optical_offset_x" value="-0.01" />
   <xacro:property name="baseline" value="${sqrt(calibration.cam1.T_cn_cnm1[0][3]**2 + calibration.cam1.T_cn_cnm1[1][3]**2 + calibration.cam1.T_cn_cnm1[2][3]**2)}"/>
+  <xacro:property name="accelerometer_stddev" value="${imu_calibration.imu0.accelerometer_noise_density * sqrt(imu_calibration.imu0.update_rate)}"/>
+  <xacro:property name="gyroscope_stddev" value="${imu_calibration.imu0.gyroscope_noise_density * sqrt(imu_calibration.imu0.update_rate)}"/>
+  <xacro:property name="accelerometer_bias_stddev" value="${imu_calibration.imu0.accelerometer_random_walk * sqrt(imu_calibration.imu0.update_rate)}"/>
+  <xacro:property name="gyroscope_bias_stddev" value="${imu_calibration.imu0.gyroscope_random_walk * sqrt(imu_calibration.imu0.update_rate)}"/>
   <link name="${prefix}_camera">
     <visual>
@@ -19,8 +23,4 @@
       </geometry>
     </collision>
-    <inertial>
-      <mass value="${cameras_inertial['oak-d-w_mass']}"/>
-      <inertia ixx="${cameras_inertial['oak-d-w_inertia']['ixx']}" ixy="${cameras_inertial['oak-d-w_inertia']['ixy']}" ixz="${cameras_inertial['oak-d-w_inertia']['ixz']}" iyy="${cameras_inertial['oak-d-w_inertia']['iyy']}" iyz="${cameras_inertial['oak-d-w_inertia']['iyz']}" izz="${cameras_inertial['oak-d-w_inertia']['izz']}"/>
-    </inertial>
   </link>
   <link name="${prefix}_rgb_camera_optical"/>
@@ -30,4 +30,5 @@
   <link name="${prefix}_right_camera"/>
   <link name="${prefix}_camera_imu_link"/>
+  <link name="${prefix}_camera_imu_link_ned"/>
   <joint name="${prefix}_rgb_camera_optical_joint" type="fixed">
     <origin xyz="${optical_offset_x} 0 0" rpy="${-pi/2} 0.0 ${-pi/2}"/>
@@ -59,4 +60,9 @@
     <parent link="${prefix}_left_camera_optical"/>
     <child link="${prefix}_camera_imu_link"/>
+  </joint>
+  <joint name="${prefix}_camera_imu_link_ned_joint" type="fixed">
+    <origin xyz="0 0 0" rpy="0 ${pi} ${-pi/2}"/>
+    <parent link="${prefix}_camera_imu_link"/>
+    <child link="${prefix}_camera_imu_link_ned"/>
   </joint>
   <!-- Stereo and depth camera -->
@@ -199,18 +205,18 @@
           <x>
             <noise type="gaussian">
-              <stddev>${imu_calibration.imu0.gyroscope_noise_density * sqrt(imu_calibration.imu0.update_rate)}</stddev>
-              <bias_stddev>${imu_calibration.imu0.gyroscope_random_walk * sqrt(imu_calibration.imu0.update_rate)}</bias_stddev>
+              <stddev>${gyroscope_stddev}</stddev>
+              <bias_stddev>${gyroscope_bias_stddev}</bias_stddev>
             </noise>
           </x>
           <y>
             <noise type="gaussian">
-              <stddev>${imu_calibration.imu0.gyroscope_noise_density * sqrt(imu_calibration.imu0.update_rate)}</stddev>
-              <bias_stddev>${imu_calibration.imu0.gyroscope_random_walk * sqrt(imu_calibration.imu0.update_rate)}</bias_stddev>
+              <stddev>${gyroscope_stddev}</stddev>
+              <bias_stddev>${gyroscope_bias_stddev}</bias_stddev>
             </noise>
           </y>
           <z>
             <noise type="gaussian">
-              <stddev>${imu_calibration.imu0.gyroscope_noise_density * sqrt(imu_calibration.imu0.update_rate)}</stddev>
-              <bias_stddev>${imu_calibration.imu0.gyroscope_random_walk * sqrt(imu_calibration.imu0.update_rate)}</bias_stddev>
+              <stddev>${gyroscope_stddev}</stddev>
+              <bias_stddev>${gyroscope_bias_stddev}</bias_stddev>
             </noise>
           </z>
@@ -219,18 +225,18 @@
           <x>
             <noise type="gaussian">
-              <stddev>${imu_calibration.imu0.accelerometer_noise_density * sqrt(imu_calibration.imu0.update_rate)}</stddev>
-              <bias_stddev>${imu_calibration.imu0.accelerometer_random_walk * sqrt(imu_calibration.imu0.update_rate)}</bias_stddev>
+              <stddev>${accelerometer_stddev}</stddev>
+              <bias_stddev>${accelerometer_bias_stddev}</bias_stddev>
             </noise>
           </x>
           <y>
             <noise type="gaussian">
-              <stddev>${imu_calibration.imu0.accelerometer_noise_density * sqrt(imu_calibration.imu0.update_rate)}</stddev>
-              <bias_stddev>${imu_calibration.imu0.accelerometer_random_walk * sqrt(imu_calibration.imu0.update_rate)}</bias_stddev>
+              <stddev>${accelerometer_stddev}</stddev>
+              <bias_stddev>${accelerometer_bias_stddev}</bias_stddev>
             </noise>
           </y>
           <z>
             <noise type="gaussian">
-              <stddev>${imu_calibration.imu0.accelerometer_noise_density * sqrt(imu_calibration.imu0.update_rate)}</stddev>
-              <bias_stddev>${imu_calibration.imu0.accelerometer_random_walk * sqrt(imu_calibration.imu0.update_rate)}</bias_stddev>
+              <stddev>${accelerometer_stddev}</stddev>
+              <bias_stddev>${accelerometer_bias_stddev}</bias_stddev>
             </noise>
           </z>
@@ -244,7 +250,7 @@
         <xyzOffset>0 0.0 0.0</xyzOffset>
         <rpyOffset>0 0 ${datum[2] * pi/180}</rpyOffset>
-        <orientationCovariance>3.5 3.5 3.5</orientationCovariance>
-        <angularVelocityCovariance>${imu_calibration.imu0.gyroscope_noise_density**2} 0 0 0 ${imu_calibration.imu0.gyroscope_noise_density**2} 0 0 0 ${imu_calibration.imu0.gyroscope_noise_density**2}</angularVelocityCovariance>
-        <linearAccelerationCovariance>${imu_calibration.imu0.accelerometer_noise_density**2} 0 0 0 ${imu_calibration.imu0.accelerometer_noise_density**2} 0 0 0 ${imu_calibration.imu0.accelerometer_noise_density**2}</linearAccelerationCovariance>
+        <orientationCovariance>0.061086523819801536 0.061086523819801536 0.061086523819801536</orientationCovariance> <!-- 3.5deg from datasheet -->
+        <angularVelocityCovariance>${gyroscope_stddev**2} ${gyroscope_stddev**2} ${gyroscope_stddev**2}</angularVelocityCovariance>
+        <linearAccelerationCovariance>${100*accelerometer_stddev**2} ${100*accelerometer_stddev**2} ${100*accelerometer_stddev**2}</linearAccelerationCovariance>
       </plugin>
     </sensor>

File: src/sirius_common/sirius_description/urdf/sirius/gnss.urdf.xacro (robot description, xacro)
@@ -3,6 +3,11 @@
      https://www.sparkfun.com/products/21801 -->
 <robot xmlns:xacro="http://wiki.ros.org/xacro">
-<xacro:macro name="gnss" params="prefix:='' material collisions:=${xacro.load_yaml('$(find sirius_description)/urdf/sirius/collisions.yaml')} inertial:=${xacro.load_yaml('$(find sirius_description)/config/inertial/gnss.yaml')} datum:=^ elevation:=^ horizontal_cep:=1.0 vertical_cep:=1.5 rate:=20.0">
+<xacro:macro name="gnss" params="prefix:='' material collisions:=${xacro.load_yaml('$(find sirius_description)/urdf/sirius/collisions.yaml')} datum:=^ elevation:=^ horizontal_cep:=1.0 vertical_cep:=1.5 rate:=20.0">
   <xacro:property name="_prefix" value="${prefix + '_' if prefix else ''}"/>
+  <!-- sqrt(-1/(2*ln(0.5))) = 0.8493218002880191 -->
+  <!-- This is the ratio needed to convert CEP to std dev of single axis -->
+  <xacro:property name="vertical_stddev" value="${vertical_cep * 0.8493218002880191}"/>
+  <xacro:property name="horizontal_stddev" value="${horizontal_cep * 0.8493218002880191}"/>
+  <xacro:property name="velocity_stddev" value="${0.05 * 0.8493218002880191}"/>
   <link name="${_prefix}gnss">
     <visual>
@@ -14,8 +19,4 @@
       <origin xyz="0 0 ${collisions['gnss_height']/2}" rpy="${pi/2} 0 0" />
     </visual>
-    <inertial>
-      <mass value="${inertial['gnss_mass']}"/>
-      <inertia ixx="${inertial['gnss_inertia']['ixx']}" ixy="${inertial['gnss_inertia']['ixy']}" ixz="${inertial['gnss_inertia']['ixz']}" iyy="${inertial['gnss_inertia']['iyy']}" iyz="${inertial['gnss_inertia']['iyz']}" izz="${inertial['gnss_inertia']['izz']}"/>
-    </inertial>
     <collision>
       <geometry>
@@ -33,13 +34,10 @@
           <horizontal>
             <noise type="gaussian">
-              <!-- sqrt(-1/(2*ln(0.5))) = 0.8493218002880191 -->
-              <!-- This is the ratio needed to convert CEP to std dev of single axis -->
-              <stddev>${horizontal_cep * 0.8493218002880191}</stddev>
+              <stddev>${horizontal_stddev}</stddev>
             </noise>
           </horizontal>
           <vertical>
             <noise type="gaussian">
-              <mean>0.0</mean>
-              <stddev>${vertical_cep * 0.8493218002880191}</stddev>
+              <stddev>${vertical_stddev}</stddev>
             </noise>
           </vertical>
@@ -48,10 +46,10 @@
           <horizontal>
             <noise type="gaussian">
-              <stddev>${0.05 * 0.8493218002880191}</stddev>
+              <stddev>${velocity_stddev}</stddev>
             </noise>
           </horizontal>
           <vertical>
             <noise type="gaussian">
-              <stddev>${0.05 * 0.8493218002880191}</stddev>
+              <stddev>${velocity_stddev}</stddev>
             </noise>
           </vertical>
@@ -68,6 +66,5 @@
             <elevation>${elevation}</elevation>
         </sphericalCoordinates>
-        <positionCovariance>${horizontal_cep * 0.8493218002880191} 0 0 0 ${horizontal_cep * 0.8493218002880191} 0 0 0 ${vertical_cep * 0.8493218002880191}</positionCovariance>
-        <positionCovarianceType>diagonal_known</positionCovarianceType>
+        <positionCovariance>${horizontal_stddev} 0 0 0 ${horizontal_stddev} 0 0 0 ${vertical_stddev}</positionCovariance>
       </plugin>
     </sensor>

File: src/sirius_common/sirius_description/urdf/sirius/indicator_light.urdf.xacro (robot description, xacro)
@@ -1,5 +1,5 @@
 <?xml version="1.0" encoding="utf-8"?>
 <robot xmlns:xacro="http://wiki.ros.org/xacro">
-<xacro:macro name="indicator_light" params="material prefix:='' collisions:=${xacro.load_yaml('$(find sirius_description)/urdf/sirius/collisions.yaml')} inertial:=${xacro.load_yaml('$(find sirius_description)/config/inertial/indicator_light.yaml')}">
+<xacro:macro name="indicator_light" params="material prefix:='' collisions:=${xacro.load_yaml('$(find sirius_description)/urdf/sirius/collisions.yaml')}">
   <xacro:property name="_prefix" value="${prefix + '_' if prefix else ''}"/>
   <link name="${_prefix}indicator_light">
@@ -11,8 +11,4 @@
       </geometry>
     </visual>
-    <inertial>
-      <mass value="${inertial['indicator_light_mass']}"/>
-      <inertia ixx="${inertial['indicator_light_inertia']['ixx']}" ixy="${inertial['indicator_light_inertia']['ixy']}" ixz="${inertial['indicator_light_inertia']['ixz']}" iyy="${inertial['indicator_light_inertia']['iyy']}" iyz="${inertial['indicator_light_inertia']['iyz']}" izz="${inertial['indicator_light_inertia']['izz']}"/>
-    </inertial>
     <collision>
       <geometry>

File: src/sirius_common/sirius_description/urdf/sirius/platform.urdf.xacro (robot description, xacro)
@@ -10,5 +10,5 @@
     </visual>
     <inertial>
-      <origin xyz="0 0 0" rpy="0 0 ${pi}"/>
+      <origin xyz="0 0 0" rpy="0 0 0"/>
       <mass value="${inertial['platform_mass']}"/>
       <inertia ixx="${inertial['platform_inertia']['ixx']}" ixy="${inertial['platform_inertia']['ixy']}" ixz="${inertial['platform_inertia']['ixz']}" iyy="${inertial['platform_inertia']['iyy']}" iyz="${inertial['platform_inertia']['iyz']}" izz="${inertial['platform_inertia']['izz']}"/>

File: src/sirius_common/sirius_description/urdf/sirius/rim.urdf.xacro (robot description, xacro)
@@ -9,11 +9,4 @@
       </geometry>
     </visual>
-    <!-- Without inertia link is either lumped with parent or removed from sdf -->
-    <!-- Link cannot be lumped with parent If we want to apply different material to it -->
-    <!-- Zero inertia is not allowed, so we use very small values as a workaround -->
-    <inertial>
-      <mass value="1e-5"/>
-      <inertia ixx="1e-9" ixy="1e-9" ixz="1e-9" iyy="1e-9" iyz="1e-9" izz="1e-9"/>
-    </inertial>
     <collision>
       <geometry>

File: src/sirius_common/sirius_description/urdf/sirius/suspension.urdf.xacro (robot description, xacro)
@@ -1,5 +1,7 @@
 <robot xmlns:xacro="http://wiki.ros.org/xacro">
-<xacro:macro name="suspension" params="prefix:='' material flip:=false mechanical:=${xacro.load_yaml('$(find sirius_description)/config/mechanical.yaml')} collisions:=${xacro.load_yaml('$(find sirius_description)/urdf/sirius/collisions.yaml')} inertial:=${xacro.load_yaml('$(find sirius_description)/config/inertial/suspension.yaml')}">
+<xacro:macro name="suspension" params="prefix:='' material flip_x_plane:=false flip_y_plane:=false mechanical:=${xacro.load_yaml('$(find sirius_description)/config/mechanical.yaml')} collisions:=${xacro.load_yaml('$(find sirius_description)/urdf/sirius/collisions.yaml')} inertial:=${xacro.load_yaml('$(find sirius_description)/config/inertial/suspension.yaml')}">
   <xacro:property name="_prefix" value="${prefix + '_' if prefix else ''}"/>
+  <xacro:property name="sign_x" value="${1 - 2 * flip_x_plane}"/>
+  <xacro:property name="sign_y" value="${1 - 2 * flip_y_plane}"/>
   <link name="${_prefix}suspension">
     <visual>
@@ -8,9 +10,10 @@
         <mesh filename="package://sirius_description/meshes/sirius/suspension.stl" scale="0.001 0.001 0.001"/>
       </geometry>
-      <origin xyz="0 0 0" rpy="0 0 ${pi if flip else 0}" />
+      <origin xyz="0 0 0" rpy="0 0 ${pi if flip_x_plane else 0}" />
     </visual>
     <inertial>
+      <origin xyz="${sign_x * inertial['suspension_center_of_mass']['x']} ${sign_y * inertial['suspension_center_of_mass']['y']} ${inertial['suspension_center_of_mass']['z']}" />
       <mass value="${inertial['suspension_mass']}"/>
-      <inertia ixx="${inertial['suspension_inertia']['ixx']}" ixy="${inertial['suspension_inertia']['ixy']}" ixz="${inertial['suspension_inertia']['ixz']}" iyy="${inertial['suspension_inertia']['iyy']}" iyz="${inertial['suspension_inertia']['iyz']}" izz="${inertial['suspension_inertia']['izz']}"/>
+      <inertia ixx="${inertial['suspension_inertia']['ixx']}" ixy="${sign_y * sign_x * inertial['suspension_inertia']['ixy']}" ixz="${sign_x * inertial['suspension_inertia']['ixz']}" iyy="${inertial['suspension_inertia']['iyy']}" iyz="${sign_y * inertial['suspension_inertia']['iyz']}" izz="${inertial['suspension_inertia']['izz']}"/>
     </inertial>
     <collision>
@@ -18,5 +21,5 @@
         <box size="${collisions['suspension_width']} ${collisions['suspension_thickness']} ${collisions['suspension_length']}"/>
       </geometry>
-      <origin xyz="${(1 - 2 * flip) * (mechanical['wheel_base']/4 - mechanical['suspension_separation_x']/4 + collisions['suspension_x_shift'])} 0 ${-mechanical['suspension_height']/2}" rpy="0 ${collisions['suspension_angle'] * pi / 180} ${pi if flip else 0}" />
+      <origin xyz="${sign_x * (mechanical['wheel_base']/4 - mechanical['suspension_separation_x']/4 + collisions['suspension_x_shift'])} 0 ${-mechanical['suspension_height']/2}" rpy="0 ${collisions['suspension_angle'] * pi / 180} ${pi if flip_x_plane else 0}" />
     </collision>
   </link>

File: src/sirius_common/sirius_description/urdf/sirius/wheel.urdf.xacro (robot description, xacro)
@@ -12,5 +12,4 @@
     </visual>
     <inertial>
-      <origin xyz="0 ${-mechanical['wheel_width']/2} 0" />
       <mass value="${inertial['wheel_mass']}"/>
       <inertia ixx="${inertial['wheel_inertia']['ixx']}" ixy="${inertial['wheel_inertia']['ixy']}" ixz="${inertial['wheel_inertia']['ixz']}" iyy="${inertial['wheel_inertia']['iyy']}" iyz="${inertial['wheel_inertia']['iyz']}" izz="${inertial['wheel_inertia']['izz']}"/>
@@ -39,13 +38,7 @@
       <xacro:element xacro:name="xacro:${material}" />
     </visual>
-  </gazebo>
-  <!-- This is required so wheel and rim link are not lumped together -->
-  <!-- Otherwise, they would be given the same material (color) during urdf->sdf conversion -->
-  <!-- Possibly, in future versions of gazebo, we could apply different materials to different visual elements in URDF -->
-  <gazebo reference="${_prefix}outer_rim_joint">
-    <preserveFixedJoint>true</preserveFixedJoint>
-  </gazebo>
-  <gazebo reference="${_prefix}inner_rim_joint">
-    <preserveFixedJoint>true</preserveFixedJoint>
+      <kd>5000.0</kd>
+      <kp>1e3</kp>
+      <max_vel>0.1</max_vel>
   </gazebo>
 </xacro:macro>
